Commit message: Update scara_robot_simple.urdf

File: scara_test_description/scara_robot_simple.urdf (robot description, URDF)
Before this commit: robot scara_robot_simple, 6 links, 5 joints
Links:
- removed link world
Joints:
- removed joint world
- joint joint1: origin xyz=0 0 0 rpy=0 0 0 -> xyz=0 0 0.2 rpy=0 0 0
- joint joint2: origin xyz=0.6 0 0 rpy=0 0 0 -> xyz=0.6 0 0.05 rpy=0 0 0
- joint joint3: limit lower=-0.1 upper=0.1 effort=10 velocity=3 -> lower=-0.08 upper=0.12 effort=10 velocity=3
- joint joint4: origin xyz=0 0 0 rpy=0 0 0 -> xyz=0 0 -0.15 rpy=0 0 0

Commit message: --joint 4 is removed from scara_robot_simple.urdf file ++vistual tags are added to scara_robot_simple.urdf file

File: scara_test_description/scara_robot_simple.urdf (robot description, URDF)
Before this commit: robot scara_robot_simple, 5 links, 4 joints
Links:
- removed link link4
- link base_link: geometry collision cylinder length=0.2 radius=0.1; visual cylinder length=0.2 radius=0.1
- link link1: geometry collision box size=0.6 0.2 0.05; visual box size=0.6 0.2 0.05
- link link2: geometry collision box size=0.4 0.2 0.05; visual box size=0.4 0.2 0.05
- link link3: geometry collision cylinder length=0.3 radius=0.02; visual cylinder length=0.3 radius=0.02
Joints:
- removed joint joint4
